File: ZigbeeZwaveEthernetadapter.kicad_sch (KiCad schematic)
At the start: 23 parts, among them J1 Barrel_Jack, J11 Conn_02x06_Odd_Even, J12 Conn_01x06, J14 Conn_01x06, J2 USB_B_Micro, J21 Conn_02x06_Odd_Even, J22 Conn_01x06, J24 Conn_01x06, J3 USB4125-GF-A, J31 Conn_02x05_Odd_Even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

Commit message: Mod: Footprint of the GCT_USB4125-GF-A, moved it to the global library.
Parts:
- J1: footprint connectors:PJ-037A -> connectors:CUI_PJ-037A
- J3: footprint ZigbeeZwaveEthernetadapter:GCT_USB4125-GF-A -> connectors:GCT_USB4125-GF-A
Changed lines of the file:
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@@
       (effects (font (size 1.27 1.27)) (justify right))
     )
-    (property "Footprint" "connectors:PJ-037A" (id 2) (at 234.95 143.256 0)
+    (property "Footprint" "connectors:CUI_PJ-037A" (id 2) (at 234.95 143.256 0)
       (effects (font (size 1.27 1.27)) hide)
     )
@@
       (effects (font (size 1.27 1.27)) (justify left))
     )
-    (property "Footprint" "ZigbeeZwaveEthernetadapter:GCT_USB4125-GF-A" (id 2) (at 241.3 49.53 0)
+    (property "Footprint" "connectors:GCT_USB4125-GF-A" (id 2) (at 241.3 49.53 0)
       (effects (font (size 1.27 1.27)) (justify bottom) hide)
     )
@@
     )
     (path "/45ccafcf-91a6-475a-88ef-bc1903af912b"
-      (reference "J1") (unit 1) (value "Barrel_Jack") (footprint "connectors:PJ-037A")
+      (reference "J1") (unit 1) (value "Barrel_Jack") (footprint "connectors:CUI_PJ-037A")
     )
     (path "/0f5191d7-13d2-4136-8d2a-cb1379a2e5b4"
@@
     )
     (path "/f71369f0-fe7d-4e5f-876d-a5b0df357ba9"
-      (reference "J3") (unit 1) (value "USB4125-GF-A") (footprint "ZigbeeZwaveEthernetadapter:GCT_USB4125-GF-A")
+      (reference "J3") (unit 1) (value "USB4125-GF-A") (footprint "connectors:GCT_USB4125-GF-A")
     )
     (path "/3b55a99d-348c-40f8-9a69-dea028a2f9d2"

Commit message: Add: PCB Layout to the project, almost finished
Parts:
- added H? (x3): MountingHole, symbol Mechanical:MountingHole
Changed lines of the file:
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@@
   (title_block
     (title "ZigbeeZwaveEthernetadapter")
-    (date "2023-01-17")
+    (date "2023-02-01")
     (rev "A")
     (company "ElektroNik Zoller")
@@
     (pin "6")
   )
+  (symbol (lib_id "Mechanical:MountingHole") (at 50.8 177.8 0) (unit 1)
+    (in_bom yes) (on_board yes) (fields_autoplaced)
+    (property "Reference" "H?" (id 0) (at 53.34 176.5299 0)
+      (effects (font (size 1.27 1.27)) (justify left))
+    )
+    (property "Value" "MountingHole" (id 1) (at 53.34 179.0699 0)
+      (effects (font (size 1.27 1.27)) (justify left))
+    )
+    (property "Footprint" "" (id 2) (at 50.8 177.8 0)
+      (effects (font (size 1.27 1.27)) hide)
+    )
+    (property "Datasheet" "~" (id 3) (at 50.8 177.8 0)
+      (effects (font (size 1.27 1.27)) hide)
+    )
+  )
   (symbol (lib_id "Regulator_Linear:TLV1117-33") (at 177.8 127 0) (mirror y) (unit 1)
     (in_bom yes) (on_board yes) (fields_autoplaced)
@@
     (pin "1")
   )
+  (symbol (lib_id "Mechanical:MountingHole") (at 25.4 177.8 0) (unit 1)
+    (in_bom yes) (on_board yes) (fields_autoplaced)
+    (property "Reference" "H?" (id 0) (at 27.94 176.5299 0)
+      (effects (font (size 1.27 1.27)) (justify left))
+    )
+    (property "Value" "MountingHole" (id 1) (at 27.94 179.0699 0)
+      (effects (font (size 1.27 1.27)) (justify left))
+    )
+    (property "Footprint" "" (id 2) (at 25.4 177.8 0)
+      (effects (font (size 1.27 1.27)) hide)
+    )
+    (property "Datasheet" "~" (id 3) (at 25.4 177.8 0)
+      (effects (font (size 1.27 1.27)) hide)
+    )
+  )
   (symbol (lib_id "power:+3V3") (at 63.5 35.56 0) (unit 1)
     (in_bom yes) (on_board yes) (fields_autoplaced)
@@
     )
     (pin "1")
+  )
+  (symbol (lib_id "Mechanical:MountingHole") (at 76.2 177.8 0) (unit 1)
+    (in_bom yes) (on_board yes) (fields_autoplaced)
+    (property "Reference" "H?" (id 0) (at 78.74 176.5299 0)
+      (effects (font (size 1.27 1.27)) (justify left))
+    )
+    (property "Value" "MountingHole" (id 1) (at 78.74 179.0699 0)
+      (effects (font (size 1.27 1.27)) (justify left))
+    )
+    (property "Footprint" "" (id 2) (at 76.2 177.8 0)
+      (effects (font (size 1.27 1.27)) hide)
+    )
+    (property "Datasheet" "~" (id 3) (at 76.2 177.8 0)
+      (effects (font (size 1.27 1.27)) hide)
+    )
   )
   (symbol (lib_id "ZigbeeZwaveEthernetadapter:USB4125-GF-A") (at 241.3 48.26 0) (unit 1)
@@
       (reference "D2") (unit 1) (value "LED") (footprint "LED_SMD:LED_0805_2012Metric_Pad1.15x1.40mm_HandSolder")
     )
+    (path "/ccce4616-cb08-4375-8528-f394c3a4aa73"
+      (reference "H?") (unit 1) (value "MountingHole") (footprint "")
+    )
+    (path "/ec3a3792-aec2-4d9f-b9b8-b952986c9164"
+      (reference "H?") (unit 1) (value "MountingHole") (footprint "")
+    )
+    (path "/f46fb497-4660-4ca1-b64c-db0b1e9f4e09"
+      (reference "H?") (unit 1) (value "MountingHole") (footprint "")
+    )
     (path "/45ccafcf-91a6-475a-88ef-bc1903af912b"

Commit message: Mod: Schematic, moved footprint to global library own
Parts:
- removed J3: USB4125-GF-A, connectors:GCT_USB4125-GF-A, symbol ZigbeeZwaveEthernetadapter:USB4125-GF-A
- added J3: USB4125-GF-A, ZigbeeZwaveEthernetadapter:GCT_USB4125-GF-A, symbol connectors:USB4125-GF-A
- gave numbers to parts that had none: 3
Connections:
- net +5V: now also J3.A9 (VBUS), J3.B9 (VBUS)
- net GND: now also J3.A12 (GND), J3.B12 (GND), J3.S1 (SHIELD)
- net at R1.1: now also J3.A5 (CC1)
- net at R2.1: now also J3.B5 (CC2)
Changed lines of the file:
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@@
   (symbol (lib_id "Mechanical:MountingHole") (at 50.8 177.8 0) (unit 1)
     (in_bom yes) (on_board yes) (fields_autoplaced)
-    (property "Reference" "H?" (id 0) (at 53.34 176.5299 0)
+    (property "Reference" "H2" (id 0) (at 53.34 176.5299 0)
       (effects (font (size 1.27 1.27)) (justify left))
     )
@@
   (symbol (lib_id "Mechanical:MountingHole") (at 25.4 177.8 0) (unit 1)
     (in_bom yes) (on_board yes) (fields_autoplaced)
-    (property "Reference" "H?" (id 0) (at 27.94 176.5299 0)
+    (property "Reference" "H1" (id 0) (at 27.94 176.5299 0)
       (effects (font (size 1.27 1.27)) (justify left))
     )
@@
     (pin "1")
   )
-  (symbol (lib_id "Mechanical:MountingHole") (at 76.2 177.8 0) (unit 1)
-    (in_bom yes) (on_board yes) (fields_autoplaced)
-    (property "Reference" "H?" (id 0) (at 78.74 176.5299 0)
-      (effects (font (size 1.27 1.27)) (justify left))
-    )
-    (property "Value" "MountingHole" (id 1) (at 78.74 179.0699 0)
-      (effects (font (size 1.27 1.27)) (justify left))
-    )
-    (property "Footprint" "" (id 2) (at 76.2 177.8 0)
-      (effects (font (size 1.27 1.27)) hide)
-    )
-    (property "Datasheet" "~" (id 3) (at 76.2 177.8 0)
-      (effects (font (size 1.27 1.27)) hide)
-    )
-  )
-  (symbol (lib_id "ZigbeeZwaveEthernetadapter:USB4125-GF-A") (at 241.3 48.26 0) (unit 1)
+  (symbol (lib_id "connectors:USB4125-GF-A") (at 241.3 48.26 0) (unit 1)
     (in_bom yes) (on_board yes)
     (property "Reference" "J3" (id 0) (at 231.14 30.48 0)
@@
       (effects (font (size 1.27 1.27)) (justify left))
     )
-    (property "Footprint" "connectors:GCT_USB4125-GF-A" (id 2) (at 241.3 49.53 0)
+    (property "Footprint" "ZigbeeZwaveEthernetadapter:GCT_USB4125-GF-A" (id 2) (at 241.3 49.53 0)
       (effects (font (size 1.27 1.27)) (justify bottom) hide)
     )
@@
     (pin "S1")
   )
+  (symbol (lib_id "Mechanical:MountingHole") (at 76.2 177.8 0) (unit 1)
+    (in_bom yes) (on_board yes) (fields_autoplaced)
+    (property "Reference" "H3" (id 0) (at 78.74 176.5299 0)
+      (effects (font (size 1.27 1.27)) (justify left))
+    )
+    (property "Value" "MountingHole" (id 1) (at 78.74 179.0699 0)
+      (effects (font (size 1.27 1.27)) (justify left))
+    )
+    (property "Footprint" "" (id 2) (at 76.2 177.8 0)
+      (effects (font (size 1.27 1.27)) hide)
+    )
+    (property "Datasheet" "~" (id 3) (at 76.2 177.8 0)
+      (effects (font (size 1.27 1.27)) hide)
+    )
+  )
   (sheet_instances
     (path "/" (page "1"))
@@
       (reference "D2") (unit 1) (value "LED") (footprint "LED_SMD:LED_0805_2012Metric_Pad1.15x1.40mm_HandSolder")
     )
+    (path "/ec3a3792-aec2-4d9f-b9b8-b952986c9164"
+      (reference "H1") (unit 1) (value "MountingHole") (footprint "")
+    )
     (path "/ccce4616-cb08-4375-8528-f394c3a4aa73"
-      (reference "H?") (unit 1) (value "MountingHole") (footprint "")
-    )
-    (path "/ec3a3792-aec2-4d9f-b9b8-b952986c9164"
-      (reference "H?") (unit 1) (value "MountingHole") (footprint "")
+      (reference "H2") (unit 1) (value "MountingHole") (footprint "")
     )
     (path "/f46fb497-4660-4ca1-b64c-db0b1e9f4e09"
-      (reference "H?") (unit 1) (value "MountingHole") (footprint "")
+      (reference "H3") (unit 1) (value "MountingHole") (footprint "")
     )
     (path "/45ccafcf-91a6-475a-88ef-bc1903af912b"
@@
       (reference "J2") (unit 1) (value "USB_B_Micro") (footprint "connectors:AMPHENOL_10118194-0001LF")
     )
-    (path "/f71369f0-fe7d-4e5f-876d-a5b0df357ba9"
-      (reference "J3") (unit 1) (value "USB4125-GF-A") (footprint "connectors:GCT_USB4125-GF-A")
+    (path "/f45b48f7-c2aa-4113-90ec-f302a0facbf0"
+      (reference "J3") (unit 1) (value "USB4125-GF-A") (footprint "ZigbeeZwaveEthernetadapter:GCT_USB4125-GF-A")
     )
     (path "/3b55a99d-348c-40f8-9a69-dea028a2f9d2"
