File: src/RaspberryPi-UART_Ethernet_Adapter.kicad_sch (KiCad schematic)
At the start: 27 parts, among them J101 Conn_02x06_Odd_Even, J102 Conn_01x06, J104 Conn_01x06, J105 Conn_02x05_Odd_Even, J106 USB4125-GF-A, J107 USB_B_Micro, J108 Barrel_Jack, U101 TLV1117-33

Commit message: Mod: Manufacturer no. & Vendor no. of J105. Changed from socket header to pin header. Close #3
Parts:
- J105: Manufacturer Part No. RS2-10-G -> PH2-10-UA; Vendor Part No. 2057-RS2-10-G-ND -> 2057-PH2-10-UA-ND

Commit message: Mod: Footprint J106, added front paste layer, closes #1. Moved logo G1 in the middle of the plane, closes #4.
Parts:
- J106: footprint Connectors_User:GCT_USB4125-GF-A -> Connector_User:GCT_USB4125-GF-A
Changed lines of the file:
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@@
 			)
 		)
-		(property "Footprint" "Connectors_User:GCT_USB4125-GF-A"
+		(property "Footprint" "Connector_User:GCT_USB4125-GF-A"
 			(at 241.3 58.42 0)
 			(effects
